File: ZigerWordClock.kicad_sch (KiCad schematic)
At the start: 33 parts, among them U1 BH1750, U10 BTF-5V-060L-B_SK9822_LED_Stri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, U11 BTF-5V-060L-B_SK9822_LED_Stri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, U12 BTF-5V-060L-B_SK9822_LED_Stri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, U13 BTF-5V-060L-B_SK9822_LED_Stri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, U14 BTF-5V-060L-B_SK9822_LED_Stri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, U15 BTF-5V-060L-B_SK9822_LED_Stri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, U16 BTF-5V-060L-B_SK9822_LED_Stri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, U17 BTF-5V-060L-B_SK9822_LED_Stri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, U18 BTF-5V-060L-B_SK9822_LED_Stri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, U19 BTF-5V-060L-B_SK9822_LED_Stri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, U2 LILYGO(R)_TTGO_T8_ESP32-S2_V1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, U20 IR-Module_38KHz, U3 BTF-5V-060L-B_SK9822_LED_Stri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, U4 LevelShifter, U5 BTF-5V-060L-B_SK9822_LED_Stri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, U6 BTF-5V-060L-B_SK9822_LED_Stri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, U7 BTF-5V-060L-B_SK9822_LED_Stri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, U8 BTF-5V-060L-B_SK9822_LED_Stri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, U9 BTF-5V-060L-B_SK9822_LED_Stri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

Commit message: first routing done
Parts:
- added J1: SAO 1.69bis, Connector_PinSocket_2.54mm:PinSocket_2x03_P2.54mm_Vertical_SMD, symbol Connector_Generic:Conn_02x03_Odd_Even
- added JP12, JP13, JP14, JP15, JP16, JP17, JP18, JP19, JP20, JP21, JP22, JP23, JP24, JP25, JP26, JP27, JP28, JP29, JP30, JP31, JP32, JP33, JP34, JP35, JP36, JP37, JP38: Pad, WordClock Footprint Library:Pad, symbol WordClock Symbol Library:Pad
Connections:
- net +3V3: now also J1.1 (Pin_1)
- net GND: now also U2.26 (GND), J1.2 (Pin_2)
- net SCL: now also J1.4 (Pin_4)
- net SDA: now also J1.3 (Pin_3)
- net at U2.10 (IO16): now also JP16.1
- net at U2.11 (IO15): now also JP17.1
- net at U2.12 (IO11): now also JP18.1
- net at U2.13 (IO12): now also JP19.1
- net at U2.14 (IO13): now also JP20.1
- net GPIO1: now reaches U2.15 (IO17)
- net GPIO1: now also J1.5 (Pin_5), JP21.1
- net GPIO2: now reaches U2.16 (IO18)
- net GPIO2: now also J1.6 (Pin_6), JP22.1
- net at U2.17 (IO20): now also JP23.1
- net at U2.18 (IO19): now also JP24.1
- net at U2.19 (VBat): now also JP25.1
- net at U2.20 (5V): now also JP26.1
- net at U2.29 (IO33): now also JP38.1
- net at U2.30 (IO34): now also JP37.1
- net at U2.31 (IO35): now also JP36.1
- net at U2.32 (IO36): now also JP35.1
- net at U2.33 (IO37): now also JP34.1
- net at U2.34 (IO38): now also JP33.1
- net at U2.35 (IO39): now also JP32.1
- net at U2.36 (IO40): now also JP31.1
- net at U2.37 (IO41): now also JP30.1
- net at U2.38 (IO42): now also JP29.1
- net at U2.39 (IO45): now also JP28.1
- net at U2.40 (IO46): now also JP27.1
- net at U2.6 (IO05): now also JP12.1
- net at U2.7 (IO06): now also JP13.1
- net at U2.8 (IO07): now also JP14.1
- net at U2.9 (IO08): now also JP15.1
