File: ZigerWordClock.kicad_pcb (KiCad board)
At the start: 2 copper layers, 237 x 237 mm, 104 parts, among them J1 SAO 1.69bis, J2 Barrel_Jack, U1 BH1750, U10 BTF-5V-060L-B_SK9822_LED_Stri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, U11 BTF-5V-060L-B_SK9822_LED_Stri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, U12 BTF-5V-060L-B_SK9822_LED_Stri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, U13 BTF-5V-060L-B_SK9822_LED_Stri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, U14 BTF-5V-060L-B_SK9822_LED_Stri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, U15 BTF-5V-060L-B_SK9822_LED_Stri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, U16 BTF-5V-060L-B_SK9822_LED_Stri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, U17 BTF-5V-060L-B_SK9822_LED_Stri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, U18 BTF-5V-060L-B_SK9822_LED_Stri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, U19 BTF-5V-060L-B_SK9822_LED_Stri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, U2 LILYGO(R)_TTGO_T8_ESP32-S2_V1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, U20 IR-Module_38KHz, U3 BTF-5V-060L-B_SK9822_LED_Stri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, U4 LevelShifter, U5 BTF-5V-060L-B_SK9822_LED_Stri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, U6 BTF-5V-060L-B_SK9822_LED_Stri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, U7 BTF-5V-060L-B_SK9822_LED_Stri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, U8 BTF-5V-060L-B_SK9822_LED_Stri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, U9 BTF-5V-060L-B_SK9822_LED_Stri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

Commit message: mounting holes fixed
Parts:
- removed the REF** at (168.5, 157.8)
- removed the REF** at (46.0, 35.2)
- removed the REF** at (146.8, 262.5)
- removed the REF** at (183.0, 39.0)
- removed the REF** at (58.0, 147.2)
- removed the REF** at (46.5, 263.5)
- removed the REF** at (260.2, 153.0)
- added REF**: MountingHole_3.2mm_M3, MountingHole:MountingHole_3.2mm_M3, F.Cu at (46.5, 263.4)

Commit message: Mouning holes fixed
Parts:
- removed the REF** at (46.5, 263.4)
- added REF**: MountingHole_3.2mm_M3, MountingHole:MountingHole_3.2mm_M3, F.Cu at (168.5, 157.8)
- added REF**: MountingHole_3.2mm_M3, MountingHole:MountingHole_3.2mm_M3, F.Cu at (46.0, 35.2)
- added REF**: MountingHole_3.2mm_M3, MountingHole:MountingHole_3.2mm_M3, F.Cu at (146.8, 262.5)
- added REF**: MountingHole_3.2mm_M3, MountingHole:MountingHole_3.2mm_M3, F.Cu at (183.0, 39.0)
- added REF**: MountingHole_3.2mm_M3, MountingHole:MountingHole_3.2mm_M3, F.Cu at (58.0, 147.2)
- added REF**: MountingHole_3.2mm_M3, MountingHole:MountingHole_3.2mm_M3, F.Cu at (46.5, 263.5)
- added REF**: MountingHole_3.2mm_M3, MountingHole:MountingHole_3.2mm_M3, F.Cu at (260.2, 153.0)
